File: microcouple/ir-transceiver.kicad_sch (KiCad schematic)
At the start: 0 parts

Commit message: Sketch out IR transceiver
Parts:
- added C10, C11: C, Capacitor_SMD:C_0805_2012Metric_Pad1.18x1.45mm_HandSolder, symbol Device:C
- added C12: 100nF, Capacitor_SMD:C_0805_2012Metric_Pad1.18x1.45mm_HandSolder, symbol Device:C
- added D65: IR, LED_THT:LED_D5.0mm_Horizontal_O1.27mm_Z3.0mm_Clear, symbol Device:LED
- added Q1: Q_Photo_NPN, LED_THT:LED_D5.0mm_Horizontal_O1.27mm_Z3.0mm, symbol Device:Q_Photo_NPN
- added R2: 5.1k, Resistor_SMD:R_0805_2012Metric_Pad1.20x1.40mm_HandSolder, symbol Device:R_US
- added R3, R4, R5: R_US, Resistor_SMD:R_0805_2012Metric_Pad1.20x1.40mm_HandSolder, symbol Device:R_US
- added R6: 180R, Resistor_SMD:R_0805_2012Metric_Pad1.20x1.40mm_HandSolder, symbol Device:R_US
- added U2: LMV358, Package_SO:SOP-8_6.605x9.655mm_P2.54mm, symbol Amplifier_Operational:LMV358
Connections:
- new net: C10.2, C11.2, R3.1, R5.1, U2.1, U2.2 (-)
- new net: R4.1, R5.2, U2.5 (+)
- new net: D65.1 (K), R6.1
- new net: C10.1, Q1.1 (C), R2.2
- new net +3.3V: C12.1, R2.1, U2.8 (V+)
- new net GND: C11.1, C12.2, Q1.2 (E), R3.2, R6.2, U2.3 (+), U2.4 (V-), U2.6 (-)
- new net IR.RX: R4.2, U2.7
- new net IR.TX: D65.2 (A)
Other:
- note added: "Collector off current = 100nA V_Roff = 510uV"
- note added: "Modulated at 38kHz NEC transmission protocol High pass filter -> schmitt trigger for demodulation"
- note added: "The op amp already rolls off higher frequency signals, so by adding a high pass filter in front we effectively create a band pass filter for the modulated signal."

Commit message: Finalize battery management
Parts:
- removed C10, C11: C, Capacitor_SMD:C_0805_2012Metric_Pad1.18x1.45mm_HandSolder, symbol Device:C
- removed C12: 100nF, Capacitor_SMD:C_0805_2012Metric_Pad1.18x1.45mm_HandSolder, symbol Device:C
- removed D65: IR, LED_THT:LED_D5.0mm_Horizontal_O1.27mm_Z3.0mm_Clear, symbol Device:LED
- removed Q1: Q_Photo_NPN, LED_THT:LED_D5.0mm_Horizontal_O1.27mm_Z3.0mm, symbol Device:Q_Photo_NPN
- removed R2: 5.1k, Resistor_SMD:R_0805_2012Metric_Pad1.20x1.40mm_HandSolder, symbol Device:R_US
- removed R3, R4, R5: R_US, Resistor_SMD:R_0805_2012Metric_Pad1.20x1.40mm_HandSolder, symbol Device:R_US
- removed R6: 180R, Resistor_SMD:R_0805_2012Metric_Pad1.20x1.40mm_HandSolder, symbol Device:R_US
- removed U2: LMV358, Package_SO:SOP-8_6.605x9.655mm_P2.54mm, symbol Amplifier_Operational:LMV358
Other:
- note removed: "Collector off current = 100nA V_Roff = 510uV"
- note removed: "Modulated at 38kHz NEC transmission protocol High pass filter -> schmitt trigger for demodulation"
- note removed: "The op amp already rolls off higher frequency signals, so by adding a high pass filter in front we effectively create a band pass filter for the modulated signal."
