File: microcouple/microcouple.kicad_pcb (KiCad board)
At the start: 2 copper layers, 0 parts

Commit message: Switch THT IR components to SMD ones
Parts:
- added BT1: 3.7V LiPo, Connector_JST:JST_PH_S2B-PH-K_1x02_P2.00mm_Horizontal, F.Cu at (89.2, 117.3)
- added C1: 100nF, Capacitor_SMD:C_0201_0603Metric, F.Cu at (95.5, 110.8)
- added C10: 14 pF, Capacitor_SMD:C_0201_0603Metric, F.Cu at (95.5, 119.5)
- added C11: 14 pF, Capacitor_SMD:C_0201_0603Metric, F.Cu at (98.0, 110.8)
- added C12: 100nF, Capacitor_SMD:C_0201_0603Metric, F.Cu at (98.0, 112.5)
- added C13: 4.7uF, Capacitor_SMD:C_0402_1005Metric, F.Cu at (115.3, 106.9)
- added C14: 4.7uF, Capacitor_SMD:C_0402_1005Metric, F.Cu at (115.3, 108.9)
- added C15: 4.7uF, Capacitor_SMD:C_0402_1005Metric, F.Cu at (115.3, 110.9)
- added C16: 4.7uF, Capacitor_SMD:C_0402_1005Metric, F.Cu at (115.3, 112.8)
- added C17: 4.7uF, Capacitor_SMD:C_0402_1005Metric, F.Cu at (106.2, 97.4)
- added C18: 100nF, Capacitor_SMD:C_0201_0603Metric, F.Cu at (103.6, 91.0)
- added C19: 100nF, Capacitor_SMD:C_0201_0603Metric, F.Cu at (103.6, 92.8)
- added C2: 100nF, Capacitor_SMD:C_0201_0603Metric, F.Cu at (95.5, 112.5)
- added C20: 100nF, Capacitor_SMD:C_0201_0603Metric, F.Cu at (114.3, 92.0)
- added C21: 100nF, Capacitor_SMD:C_0201_0603Metric, F.Cu at (114.3, 93.7)
- added C22: 100nF, Capacitor_SMD:C_0201_0603Metric, F.Cu at (120.5, 86.5)
- added C23: 100nF, Capacitor_SMD:C_0201_0603Metric, F.Cu at (112.7, 106.8)
- added C3: 100nF, Capacitor_SMD:C_0201_0603Metric, F.Cu at (95.5, 114.3)
- added C4: 4.7uF, Capacitor_SMD:C_0402_1005Metric, F.Cu at (107.8, 101.4)
- added C5: 4.7uF, Capacitor_SMD:C_0402_1005Metric, F.Cu at (107.8, 103.3)
- added C6: 100nF, Capacitor_SMD:C_0201_0603Metric, F.Cu at (95.5, 116.0)
- added C7: 4.7uF, Capacitor_SMD:C_0402_1005Metric, F.Cu at (107.8, 105.3)
- added C8: 100nF, Capacitor_SMD:C_0201_0603Metric, F.Cu at (95.5, 117.8)
- added C9: 4.7uF, Capacitor_SMD:C_0402_1005Metric, F.Cu at (107.8, 107.3)
- added D1: GREEN, LED_SMD:LED_0201_0603Metric, F.Cu at (108.2, 121.2)
- added D10: RED, LED_SMD:LED_0201_0603Metric, F.Cu at (87.7, 88.5)
- added D11: RED, LED_SMD:LED_0201_0603Metric, F.Cu at (87.7, 90.3)
- added D12: RED, LED_SMD:LED_0201_0603Metric, F.Cu at (87.7, 92.0)
- added D13: RED, LED_SMD:LED_0201_0603Metric, F.Cu at (87.7, 93.8)
- added D14: RED, LED_SMD:LED_0201_0603Metric, F.Cu at (87.7, 95.5)
- added D15: RED, LED_SMD:LED_0201_0603Metric, F.Cu at (87.7, 97.3)
- added D16: RED, LED_SMD:LED_0201_0603Metric, F.Cu at (90.4, 79.8)
- added D17: RED, LED_SMD:LED_0201_0603Metric, F.Cu at (90.4, 81.5)
- added D18: RED, LED_SMD:LED_0201_0603Metric, F.Cu at (90.4, 83.3)
- added D19: RED, LED_SMD:LED_0201_0603Metric, F.Cu at (90.4, 85.0)
- added D2: Charging, LED_SMD:LED_0201_0603Metric, F.Cu at (115.4, 114.7)
- added D20: RED, LED_SMD:LED_0201_0603Metric, F.Cu at (90.4, 86.8)
- added D21: RED, LED_SMD:LED_0201_0603Metric, F.Cu at (90.4, 88.5)
- added D22: RED, LED_SMD:LED_0201_0603Metric, F.Cu at (90.4, 90.3)
- added D23: RED, LED_SMD:LED_0201_0603Metric, F.Cu at (90.4, 92.0)
- added D24: RED, LED_SMD:LED_0201_0603Metric, F.Cu at (90.4, 93.8)
- added D25: RED, LED_SMD:LED_0201_0603Metric, F.Cu at (90.4, 95.5)
- added D26: RED, LED_SMD:LED_0201_0603Metric, F.Cu at (90.4, 97.3)
- added D27: RED, LED_SMD:LED_0201_0603Metric, F.Cu at (93.1, 79.8)
- added D28: RED, LED_SMD:LED_0201_0603Metric, F.Cu at (93.1, 81.5)
- added D29: RED, LED_SMD:LED_0201_0603Metric, F.Cu at (93.1, 83.3)
- added D3: Done, LED_SMD:LED_0201_0603Metric, F.Cu at (115.4, 116.4)
- added D30: RED, LED_SMD:LED_0201_0603Metric, F.Cu at (93.1, 85.0)
- added D31: RED, LED_SMD:LED_0201_0603Metric, F.Cu at (93.1, 86.8)
- added D32: RED, LED_SMD:LED_0201_0603Metric, F.Cu at (93.1, 88.5)
- added D33: RED, LED_SMD:LED_0201_0603Metric, F.Cu at (93.1, 90.3)
- added D34: RED, LED_SMD:LED_0201_0603Metric, F.Cu at (93.1, 92.0)
- added D35: RED, LED_SMD:LED_0201_0603Metric, F.Cu at (93.1, 93.8)
- added D36: RED, LED_SMD:LED_0201_0603Metric, F.Cu at (93.1, 95.5)
- added D37: RED, LED_SMD:LED_0201_0603Metric, F.Cu at (93.1, 97.3)
- added D38: RED, LED_SMD:LED_0201_0603Metric, F.Cu at (95.7, 79.8)
- added D39: RED, LED_SMD:LED_0201_0603Metric, F.Cu at (95.7, 81.5)
- added D4: SB5H100, Diode_SMD:D_SMB, F.Cu at (116.7, 103.2)
- added D40: RED, LED_SMD:LED_0201_0603Metric, F.Cu at (95.7, 83.3)
- added D41: RED, LED_SMD:LED_0201_0603Metric, F.Cu at (95.7, 85.0)
- added D42: RED, LED_SMD:LED_0201_0603Metric, F.Cu at (95.7, 86.8)
- added D43: RED, LED_SMD:LED_0201_0603Metric, F.Cu at (95.7, 88.5)
- added D44: RED, LED_SMD:LED_0201_0603Metric, F.Cu at (95.7, 90.3)
- added D45: RED, LED_SMD:LED_0201_0603Metric, F.Cu at (95.7, 92.0)
- added D46: RED, LED_SMD:LED_0201_0603Metric, F.Cu at (95.7, 93.8)
- added D47: RED, LED_SMD:LED_0201_0603Metric, F.Cu at (95.7, 95.5)
- added D48: RED, LED_SMD:LED_0201_0603Metric, F.Cu at (95.7, 97.3)
- added D49: RED, LED_SMD:LED_0201_0603Metric, F.Cu at (98.4, 79.8)
- added D5: RED, LED_SMD:LED_0201_0603Metric, F.Cu at (87.7, 79.8)
- added D50: RED, LED_SMD:LED_0201_0603Metric, F.Cu at (98.4, 81.5)
- added D51: RED, LED_SMD:LED_0201_0603Metric, F.Cu at (98.4, 83.3)
- added D52: RED, LED_SMD:LED_0201_0603Metric, F.Cu at (98.4, 85.0)
- added D53: RED, LED_SMD:LED_0201_0603Metric, F.Cu at (98.4, 86.8)
- added D54: RED, LED_SMD:LED_0201_0603Metric, F.Cu at (98.4, 88.5)
- added D55: RED, LED_SMD:LED_0201_0603Metric, F.Cu at (98.4, 90.3)
- added D56: RED, LED_SMD:LED_0201_0603Metric, F.Cu at (98.4, 92.0)
- added D57: RED, LED_SMD:LED_0201_0603Metric, F.Cu at (98.4, 93.8)
- added D58: RED, LED_SMD:LED_0201_0603Metric, F.Cu at (98.4, 95.5)
- added D59: RED, LED_SMD:LED_0201_0603Metric, F.Cu at (98.4, 97.3)
- added D6: RED, LED_SMD:LED_0201_0603Metric, F.Cu at (87.7, 81.5)
- added D60: RED, LED_SMD:LED_0201_0603Metric, F.Cu at (101.1, 79.8)
- added D61: RED, LED_SMD:LED_0201_0603Metric, F.Cu at (101.1, 81.5)
- added D62: RED, LED_SMD:LED_0201_0603Metric, F.Cu at (101.1, 83.3)
- added D63: RED, LED_SMD:LED_0201_0603Metric, F.Cu at (101.1, 85.0)
- added D64: RED, LED_SMD:LED_0201_0603Metric, F.Cu at (101.1, 86.8)
- added D65: RED, LED_SMD:LED_0201_0603Metric, F.Cu at (101.1, 88.5)
- added D66: RED, LED_SMD:LED_0201_0603Metric, F.Cu at (101.1, 90.3)
- added D67: RED, LED_SMD:LED_0201_0603Metric, F.Cu at (101.1, 92.0)
- added D68: RED, LED_SMD:LED_0201_0603Metric, F.Cu at (101.1, 93.8)
- added D69: IR, LED_THT:LED_SideEmitter_Rectangular_W4.5mm_H1.6mm, F.Cu at (194.5, 106.5)
- added D7: RED, LED_SMD:LED_0201_0603Metric, F.Cu at (87.7, 83.3)
- added D8: RED, LED_SMD:LED_0201_0603Metric, F.Cu at (87.7, 85.0)
- added D9: RED, LED_SMD:LED_0201_0603Metric, F.Cu at (87.7, 86.8)
- added FB1: 120R @ 100MHz, Inductor_SMD:L_0805_2012Metric_Pad1.15x1.40mm_HandSolder, F.Cu at (96.7, 121.9)
- added J1: Conn_ARM_SWD_TagConnect_TC2030-NL, Connector:Tag-Connect_TC2030-IDC-NL_2x03_P1.27mm_Vertical, F.Cu at (90.2, 112.4)
- added L1: 2.2uH, Inductor_SMD:L_1008_2520Metric, F.Cu at (126.8, 107.8)
- added P1: USB_C_Plug, GS_Connectors:USB-C-SMD, F.Cu at (91.8, 104.0)
- added Q1: AO3415, Package_TO_SOT_SMD:SOT-23_Handsoldering, F.Cu at (125.2, 102.9)
- added R1: 1k, Resistor_SMD:R_0201_0603Metric, F.Cu at (98.0, 114.3)
- added R10: 1.5k, Resistor_SMD:R_0201_0603Metric, F.Cu at (112.7, 112.1)
- added R11: 100k, Resistor_SMD:R_0201_0603Metric, F.Cu at (112.7, 113.8)
- added R12: 100k, Resistor_SMD:R_0201_0603Metric, F.Cu at (103.6, 94.5)
- added R13: 10k, Resistor_SMD:R_0201_0603Metric, F.Cu at (103.6, 96.3)
- added R14: 10k, Resistor_SMD:R_0201_0603Metric, F.Cu at (114.3, 95.5)
- added R15: 100k, Resistor_SMD:R_0201_0603Metric, F.Cu at (114.3, 97.2)
- added R16: 330R, Resistor_SMD:R_0201_0603Metric, F.Cu at (120.5, 88.2)
- added R2: 5.1k, Resistor_SMD:R_0201_0603Metric, F.Cu at (98.0, 116.0)
- added R3: 5.1k, Resistor_SMD:R_0201_0603Metric, F.Cu at (98.0, 117.8)
- added R4: 5.1k, Resistor_SMD:R_0201_0603Metric, F.Cu at (98.0, 119.5)
- added R5: 27R, Resistor_SMD:R_0201_0603Metric, F.Cu at (100.4, 110.8)
- added R6: 27R, Resistor_SMD:R_0201_0603Metric, F.Cu at (100.4, 112.5)
- added R7: 5.1k, Resistor_SMD:R_0201_0603Metric, F.Cu at (100.4, 114.3)
- added R8: 1.5k, Resistor_SMD:R_0201_0603Metric, F.Cu at (112.7, 108.6)
- added R9: 10k, Resistor_SMD:R_0201_0603Metric, F.Cu at (112.7, 110.3)
- added SW1: ~{RESET}, Button_Switch_SMD:SW_SPST_PTS810, F.Cu at (105.0, 112.3)
- added SW2: SW_SPDT_MSK12CO2, GS_Switches:MSK12CO2, F.Cu at (185.9, 120.2)
- added U1: USBLC6-2SC6, Package_TO_SOT_SMD:SOT-23-6, F.Cu at (104.2, 122.7)
- added U2: RP2040, Package_DFN_QFN:QFN-56-1EP_7x7mm_P0.4mm_EP3.2x3.2mm, F.Cu at (101.7, 105.0)
- added U3: MCP73831-2-OT, Package_TO_SOT_SMD:SOT-23-5, F.Cu at (126.7, 115.0)
- added U4: LM3671MFX, Package_TO_SOT_SMD:TSOT-23-5, F.Cu at (121.5, 114.5)
- added U6: IS31FL3729, Package_DFN_QFN:QFN-32-1EP_4x4mm_P0.4mm_EP2.65x2.65mm, F.Cu at (107.9, 93.3)
- added U7: CAP1188, Package_DFN_QFN:QFN-24-1EP_4x4mm_P0.5mm_EP2.5x2.5mm, F.Cu at (118.7, 94.2)
- added U8: TSOP34138, OptoDevice:Vishay_MOLD-3Pin, F.Cu at (193.7, 100.5)
- added X1: 12MHz 12pF, Crystal:Crystal_SMD_3225-4Pin_3.2x2.5mm, F.Cu at (105.0, 117.5)
