File: microcouple/led-matrix.kicad_sch (KiCad schematic)
At the start: 0 parts

Commit message: Sketch out IR transceiver
Parts:
- added D1, D10, D11, D12, D13, D14, D15, D16, D17, D18, D19, D2, D20, D21, D22, D23, D24, D25, D26, D27, D28, D29, D3, D30, D31, D32, D33, D34, D35, D36, D37, D38, D39, D4, D40, D41, D42, D43, D44, D45, D46, D47, D48, D49, D5, D50, D51, D52, D53, D54, D55, D56, D57, D58, D59, D6, D60, D61, D62, D63, D64, D7, D8, D9: RED, LED_SMD:LED_0805_2012Metric_Pad1.15x1.40mm_HandSolder, symbol Device:LED_45deg
Connections:
- new net: D11.1 (K), D19.1 (K), D27.1 (K), D3.1 (K), D35.1 (K), D43.1 (K), D51.1 (K), D59.1 (K)
- new net: D17.2 (A), D18.2 (A), D19.2 (A), D20.2 (A), D21.2 (A), D22.2 (A), D23.2 (A), D24.2 (A)
- new net: D16.1 (K), D24.1 (K), D32.1 (K), D40.1 (K), D48.1 (K), D56.1 (K), D64.1 (K), D8.1 (K)
- new net: D41.2 (A), D42.2 (A), D43.2 (A), D44.2 (A), D45.2 (A), D46.2 (A), D47.2 (A), D48.2 (A)
- new net: D1.2 (A), D2.2 (A), D3.2 (A), D4.2 (A), D5.2 (A), D6.2 (A), D7.2 (A), D8.2 (A)
- new net: D10.1 (K), D18.1 (K), D2.1 (K), D26.1 (K), D34.1 (K), D42.1 (K), D50.1 (K), D58.1 (K)
- new net: D13.1 (K), D21.1 (K), D29.1 (K), D37.1 (K), D45.1 (K), D5.1 (K), D53.1 (K), D61.1 (K)
- new net: D25.2 (A), D26.2 (A), D27.2 (A), D28.2 (A), D29.2 (A), D30.2 (A), D31.2 (A), D32.2 (A)
- new net: D12.1 (K), D20.1 (K), D28.1 (K), D36.1 (K), D4.1 (K), D44.1 (K), D52.1 (K), D60.1 (K)
- new net: D49.2 (A), D50.2 (A), D51.2 (A), D52.2 (A), D53.2 (A), D54.2 (A), D55.2 (A), D56.2 (A)
- new net: D15.1 (K), D23.1 (K), D31.1 (K), D39.1 (K), D47.1 (K), D55.1 (K), D63.1 (K), D7.1 (K)
- new net: D57.2 (A), D58.2 (A), D59.2 (A), D60.2 (A), D61.2 (A), D62.2 (A), D63.2 (A), D64.2 (A)
- new net: D1.1 (K), D17.1 (K), D25.1 (K), D33.1 (K), D41.1 (K), D49.1 (K), D57.1 (K), D9.1 (K)
- new net: D33.2 (A), D34.2 (A), D35.2 (A), D36.2 (A), D37.2 (A), D38.2 (A), D39.2 (A), D40.2 (A)
- new net: D10.2 (A), D11.2 (A), D12.2 (A), D13.2 (A), D14.2 (A), D15.2 (A), D16.2 (A), D9.2 (A)
- new net: D14.1 (K), D22.1 (K), D30.1 (K), D38.1 (K), D46.1 (K), D54.1 (K), D6.1 (K), D62.1 (K)

Commit message: Sketch out LED matrix
Parts:
- added C13, C14: 100nF, Capacitor_SMD:C_0805_2012Metric_Pad1.18x1.45mm_HandSolder, symbol Device:C
- added R10, R11, R12, R13, R14, R7, R8, R9: 120R, Resistor_SMD:R_0805_2012Metric_Pad1.20x1.40mm_HandSolder, symbol Device:R_US
- added U3, U4: 74HC595, Package_SO:SOIC-16_3.9x9.9mm_P1.27mm, symbol 74xx:74HC595
Connections:
- net at D11.1 (K), D19.1 (K), D27.1 (K)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: now also R9.1
- net LEDMTX.R5: now reaches D17.2 (A), D18.2 (A), D19.2 (A), D20.2 (A), D21.2 (A), D22.2 (A), D23.2 (A), D24.2 (A)
- net at D16.1 (K), D24.1 (K), D32.1 (K)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: now also R14.1
- net LEDMTX.R2: now reaches D41.2 (A), D42.2 (A), D43.2 (A), D44.2 (A), D45.2 (A), D46.2 (A), D47.2 (A), D48.2 (A)
- net LEDMTX.R7: now reaches D1.2 (A), D2.2 (A), D3.2 (A), D4.2 (A), D5.2 (A), D6.2 (A), D7.2 (A), D8.2 (A)
- net at D10.1 (K), D18.1 (K), D2.1 (K)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: now also R8.1
- net at D13.1 (K), D21.1 (K), D29.1 (K)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: now also R11.1
- net LEDMTX.R4: now reaches D25.2 (A), D26.2 (A), D27.2 (A), D28.2 (A), D29.2 (A), D30.2 (A), D31.2 (A), D32.2 (A)
- net at D12.1 (K), D20.1 (K), D28.1 (K)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: now also R10.1
- net LEDMTX.R1: now reaches D49.2 (A), D50.2 (A), D51.2 (A), D52.2 (A), D53.2 (A), D54.2 (A), D55.2 (A), D56.2 (A)
- net at D15.1 (K), D23.1 (K), D31.1 (K)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: now also R13.1
- net LEDMTX.R0: now reaches D57.2 (A), D58.2 (A), D59.2 (A), D60.2 (A), D61.2 (A), D62.2 (A), D63.2 (A), D64.2 (A)
- net at D1.1 (K), D17.1 (K), D25.1 (K)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: now also R7.1
- net LEDMTX.R3: now reaches D33.2 (A), D34.2 (A), D35.2 (A), D36.2 (A), D37.2 (A), D38.2 (A), D39.2 (A), D40.2 (A)
- net LEDMTX.R6: now reaches D10.2 (A), D11.2 (A), D12.2 (A), D13.2 (A), D14.2 (A), D15.2 (A), D16.2 (A), D9.2 (A)
- net at D14.1 (K), D22.1 (K), D30.1 (K)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: now also R12.1
- new net +3.3V: C13.1, C14.1, U3.16 (VCC), U4.16 (VCC)
- new net GND: C13.2, C14.2, U3.8 (GND), U4.8 (GND)
- new net LEDMTX.C0: R7.2
- new net LEDMTX.C1: R8.2
- new net LEDMTX.C2: R9.2
- new net LEDMTX.C3: R10.2
- new net LEDMTX.C4: R11.2
- new net LEDMTX.C5: R12.2
- new net LEDMTX.C6: R13.2
- new net LEDMTX.C7: R14.2
Other:
- note added: "Each LED runs at 8mA max current at any time = 64mA Max current sourcing/sinking by 74HC595 = 70mA No need for darlington array"
- moved on the sheet: D1, D10, D11, D12, D13, D14, D15, D16, D17, D18, D19, D2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

Commit message: First draft of LED matrix
Connections:
- net LEDMTX.C0: now also U4.15 (QA)
- net LEDMTX.C1: now also U4.1 (QB)
- net LEDMTX.C2: now also U4.2 (QC)
- net LEDMTX.C3: now also U4.3 (QD)
- net LEDMTX.C4: now also U4.4 (QE)
- net LEDMTX.C5: now also U4.5 (QF)
- net LEDMTX.C6: now also U4.6 (QG)
- net LEDMTX.C7: now also U4.7 (QH)
- net LEDMTX.R0: now also U3.15 (QA)
- net LEDMTX.R1: now also U3.1 (QB)
- net LEDMTX.R2: now also U3.2 (QC)
- net LEDMTX.R3: now also U3.3 (QD)
- net LEDMTX.R4: now also U3.4 (QE)
- net LEDMTX.R5: now also U3.5 (QF)
- net LEDMTX.R6: now also U3.6 (QG)
- net LEDMTX.R7: now also U3.7 (QH)
- net ~{SCL}: now reaches U3.10 (~{SRCLR})
- net ~{SCL}: now also U4.10 (~{SRCLR})
- net SCK: now reaches U3.11 (SRCLK)
- net SCK: now also U4.11 (SRCLK)
- net RCK: now reaches U3.12 (RCLK)
- net RCK: now also U4.12 (RCLK)
- net ~{OE}: now reaches U3.13 (~{OE})
- net ~{OE}: now also U4.13 (~{OE})
- net RSI: now reaches U3.14 (SER)
- net CSI: now reaches U4.14 (SER)
- no-connect marks 0 -> 2
Other:
- moved on the sheet: C13, C14, D1, D10, D11, D12, D13, D14, D15, D16, D17, D18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

Commit message: Finalize battery management
Parts:
- removed C13, C14: 100nF, Capacitor_SMD:C_0805_2012Metric_Pad1.18x1.45mm_HandSolder, symbol Device:C
- removed R10, R11, R12, R13, R14, R7, R8, R9: 120R, Resistor_SMD:R_0805_2012Metric_Pad1.20x1.40mm_HandSolder, symbol Device:R_US
- removed U3, U4: 74HC595, Package_SO:SOIC-16_3.9x9.9mm_P1.27mm, symbol 74xx:74HC595
- added U3 (x2): TLC59116, Package_SO:TSSOP-28_4.4x9.7mm_P0.65mm, symbol GS_IC:TLC59116
Connections:
- net +3.3V: now also U3.28 (VCC)
- net GND: now also U3.10 (GND), U3.19 (GND), U3.24 (GND)
- net LEDMTX.C0: now also D1.1 (K), D17.1 (K), D25.1 (K), D33.1 (K), D41.1 (K), D49.1 (K), D57.1 (K), D9.1 (K)
- net LEDMTX.C1: now also D10.1 (K), D18.1 (K), D2.1 (K), D26.1 (K), D34.1 (K), D42.1 (K), D50.1 (K), D58.1 (K)
- net LEDMTX.C2: now also D11.1 (K), D19.1 (K), D27.1 (K), D3.1 (K), D35.1 (K), D43.1 (K), D51.1 (K), D59.1 (K)
- net LEDMTX.C3: now also D12.1 (K), D20.1 (K), D28.1 (K), D36.1 (K), D4.1 (K), D44.1 (K), D52.1 (K), D60.1 (K)
- net LEDMTX.C4: now also D13.1 (K), D21.1 (K), D29.1 (K), D37.1 (K), D45.1 (K), D5.1 (K), D53.1 (K), D61.1 (K)
- net LEDMTX.C5: now also D14.1 (K), D22.1 (K), D30.1 (K), D38.1 (K), D46.1 (K), D54.1 (K), D6.1 (K), D62.1 (K)
- net LEDMTX.C6: now also D15.1 (K), D23.1 (K), D31.1 (K), D39.1 (K), D47.1 (K), D55.1 (K), D63.1 (K), D7.1 (K)
- net LEDMTX.C7: now also D16.1 (K), D24.1 (K), D32.1 (K), D40.1 (K), D48.1 (K), D56.1 (K), D64.1 (K), D8.1 (K)
- no-connect marks 2 -> 0
Other:
- note removed: "Each LED runs at 8mA max current at any time = 64mA Max current sourcing/sinking by 74HC595 = 70mA No need for darlington array"

Commit message: Preliminary Schematic
Parts:
- removed U3: TLC59116, Package_SO:TSSOP-28_4.4x9.7mm_P0.65mm, symbol GS_IC:TLC59116
- added C17, C19: 100nF, Capacitor_SMD:C_0201_0603Metric, symbol Device:C
- added C18: 4.7uF, Capacitor_SMD:C_0402_1005Metric, symbol Device:C
- added R12: 10k, Resistor_SMD:R_0201_0603Metric, symbol Device:R_US
- added R13: 100k, Resistor_SMD:R_0201_0603Metric, symbol Device:R_US
- added U3: IS31FL3729, Package_DFN_QFN:QFN-32-1EP_4x4mm_P0.4mm_EP2.65x2.65mm, symbol GS_LED_Drivers:IS31FL3729
- D10: renamed from D9; footprint LED_SMD:LED_0805_2012Metric_Pad1.15x1.40mm_HandSolder -> LED_SMD:LED_0201_0603Metric
- D11: renamed from D10; footprint LED_SMD:LED_0805_2012Metric_Pad1.15x1.40mm_HandSolder -> LED_SMD:LED_0201_0603Metric
- D12: renamed from D11; footprint LED_SMD:LED_0805_2012Metric_Pad1.15x1.40mm_HandSolder -> LED_SMD:LED_0201_0603Metric
- D13: renamed from D12; footprint LED_SMD:LED_0805_2012Metric_Pad1.15x1.40mm_HandSolder -> LED_SMD:LED_0201_0603Metric
- D14: renamed from D13; footprint LED_SMD:LED_0805_2012Metric_Pad1.15x1.40mm_HandSolder -> LED_SMD:LED_0201_0603Metric
- D15: renamed from D14; footprint LED_SMD:LED_0805_2012Metric_Pad1.15x1.40mm_HandSolder -> LED_SMD:LED_0201_0603Metric
- D16: renamed from D15; footprint LED_SMD:LED_0805_2012Metric_Pad1.15x1.40mm_HandSolder -> LED_SMD:LED_0201_0603Metric
- D17: renamed from D16; footprint LED_SMD:LED_0805_2012Metric_Pad1.15x1.40mm_HandSolder -> LED_SMD:LED_0201_0603Metric
- D18: renamed from D17; footprint LED_SMD:LED_0805_2012Metric_Pad1.15x1.40mm_HandSolder -> LED_SMD:LED_0201_0603Metric
- D19: renamed from D18; footprint LED_SMD:LED_0805_2012Metric_Pad1.15x1.40mm_HandSolder -> LED_SMD:LED_0201_0603Metric
- D2: renamed from D1; footprint LED_SMD:LED_0805_2012Metric_Pad1.15x1.40mm_HandSolder -> LED_SMD:LED_0201_0603Metric
- D20: renamed from D19; footprint LED_SMD:LED_0805_2012Metric_Pad1.15x1.40mm_HandSolder -> LED_SMD:LED_0201_0603Metric
- D21: renamed from D20; footprint LED_SMD:LED_0805_2012Metric_Pad1.15x1.40mm_HandSolder -> LED_SMD:LED_0201_0603Metric
- D22: renamed from D21; footprint LED_SMD:LED_0805_2012Metric_Pad1.15x1.40mm_HandSolder -> LED_SMD:LED_0201_0603Metric
- D23: renamed from D22; footprint LED_SMD:LED_0805_2012Metric_Pad1.15x1.40mm_HandSolder -> LED_SMD:LED_0201_0603Metric
- D24: renamed from D23; footprint LED_SMD:LED_0805_2012Metric_Pad1.15x1.40mm_HandSolder -> LED_SMD:LED_0201_0603Metric
- D25: renamed from D24; footprint LED_SMD:LED_0805_2012Metric_Pad1.15x1.40mm_HandSolder -> LED_SMD:LED_0201_0603Metric
- D26: renamed from D25; footprint LED_SMD:LED_0805_2012Metric_Pad1.15x1.40mm_HandSolder -> LED_SMD:LED_0201_0603Metric
- D27: renamed from D26; footprint LED_SMD:LED_0805_2012Metric_Pad1.15x1.40mm_HandSolder -> LED_SMD:LED_0201_0603Metric
- D28: renamed from D27; footprint LED_SMD:LED_0805_2012Metric_Pad1.15x1.40mm_HandSolder -> LED_SMD:LED_0201_0603Metric
- D29: renamed from D28; footprint LED_SMD:LED_0805_2012Metric_Pad1.15x1.40mm_HandSolder -> LED_SMD:LED_0201_0603Metric
- D3: renamed from D2; footprint LED_SMD:LED_0805_2012Metric_Pad1.15x1.40mm_HandSolder -> LED_SMD:LED_0201_0603Metric
- D30: renamed from D29; footprint LED_SMD:LED_0805_2012Metric_Pad1.15x1.40mm_HandSolder -> LED_SMD:LED_0201_0603Metric
- D31: renamed from D30; footprint LED_SMD:LED_0805_2012Metric_Pad1.15x1.40mm_HandSolder -> LED_SMD:LED_0201_0603Metric
- D32: renamed from D31; footprint LED_SMD:LED_0805_2012Metric_Pad1.15x1.40mm_HandSolder -> LED_SMD:LED_0201_0603Metric
- D33: renamed from D32; footprint LED_SMD:LED_0805_2012Metric_Pad1.15x1.40mm_HandSolder -> LED_SMD:LED_0201_0603Metric
- D34: renamed from D33; footprint LED_SMD:LED_0805_2012Metric_Pad1.15x1.40mm_HandSolder -> LED_SMD:LED_0201_0603Metric
- D35: renamed from D34; footprint LED_SMD:LED_0805_2012Metric_Pad1.15x1.40mm_HandSolder -> LED_SMD:LED_0201_0603Metric
- D36: renamed from D35; footprint LED_SMD:LED_0805_2012Metric_Pad1.15x1.40mm_HandSolder -> LED_SMD:LED_0201_0603Metric
- D37: renamed from D36; footprint LED_SMD:LED_0805_2012Metric_Pad1.15x1.40mm_HandSolder -> LED_SMD:LED_0201_0603Metric
- D38: renamed from D37; footprint LED_SMD:LED_0805_2012Metric_Pad1.15x1.40mm_HandSolder -> LED_SMD:LED_0201_0603Metric
- D39: renamed from D38; footprint LED_SMD:LED_0805_2012Metric_Pad1.15x1.40mm_HandSolder -> LED_SMD:LED_0201_0603Metric
- D4: renamed from D3; footprint LED_SMD:LED_0805_2012Metric_Pad1.15x1.40mm_HandSolder -> LED_SMD:LED_0201_0603Metric
- D40: renamed from D39; footprint LED_SMD:LED_0805_2012Metric_Pad1.15x1.40mm_HandSolder -> LED_SMD:LED_0201_0603Metric
- D41: renamed from D40; footprint LED_SMD:LED_0805_2012Metric_Pad1.15x1.40mm_HandSolder -> LED_SMD:LED_0201_0603Metric
- D42: renamed from D41; footprint LED_SMD:LED_0805_2012Metric_Pad1.15x1.40mm_HandSolder -> LED_SMD:LED_0201_0603Metric
- D43: renamed from D42; footprint LED_SMD:LED_0805_2012Metric_Pad1.15x1.40mm_HandSolder -> LED_SMD:LED_0201_0603Metric
- D44: renamed from D43; footprint LED_SMD:LED_0805_2012Metric_Pad1.15x1.40mm_HandSolder -> LED_SMD:LED_0201_0603Metric
- D45: renamed from D44; footprint LED_SMD:LED_0805_2012Metric_Pad1.15x1.40mm_HandSolder -> LED_SMD:LED_0201_0603Metric
- D46: renamed from D45; footprint LED_SMD:LED_0805_2012Metric_Pad1.15x1.40mm_HandSolder -> LED_SMD:LED_0201_0603Metric
- D47: renamed from D46; footprint LED_SMD:LED_0805_2012Metric_Pad1.15x1.40mm_HandSolder -> LED_SMD:LED_0201_0603Metric
- D48: renamed from D47; footprint LED_SMD:LED_0805_2012Metric_Pad1.15x1.40mm_HandSolder -> LED_SMD:LED_0201_0603Metric
- D49: renamed from D48; footprint LED_SMD:LED_0805_2012Metric_Pad1.15x1.40mm_HandSolder -> LED_SMD:LED_0201_0603Metric
- D5: renamed from D4; footprint LED_SMD:LED_0805_2012Metric_Pad1.15x1.40mm_HandSolder -> LED_SMD:LED_0201_0603Metric
- D50: renamed from D49; footprint LED_SMD:LED_0805_2012Metric_Pad1.15x1.40mm_HandSolder -> LED_SMD:LED_0201_0603Metric
- D51: renamed from D50; footprint LED_SMD:LED_0805_2012Metric_Pad1.15x1.40mm_HandSolder -> LED_SMD:LED_0201_0603Metric
- D52: renamed from D51; footprint LED_SMD:LED_0805_2012Metric_Pad1.15x1.40mm_HandSolder -> LED_SMD:LED_0201_0603Metric
- D53: renamed from D52; footprint LED_SMD:LED_0805_2012Metric_Pad1.15x1.40mm_HandSolder -> LED_SMD:LED_0201_0603Metric
- D54: renamed from D53; footprint LED_SMD:LED_0805_2012Metric_Pad1.15x1.40mm_HandSolder -> LED_SMD:LED_0201_0603Metric
- D55: renamed from D54; footprint LED_SMD:LED_0805_2012Metric_Pad1.15x1.40mm_HandSolder -> LED_SMD:LED_0201_0603Metric
- D56: renamed from D55; footprint LED_SMD:LED_0805_2012Metric_Pad1.15x1.40mm_HandSolder -> LED_SMD:LED_0201_0603Metric
- D57: renamed from D56; footprint LED_SMD:LED_0805_2012Metric_Pad1.15x1.40mm_HandSolder -> LED_SMD:LED_0201_0603Metric
- D58: renamed from D57; footprint LED_SMD:LED_0805_2012Metric_Pad1.15x1.40mm_HandSolder -> LED_SMD:LED_0201_0603Metric
- D59: renamed from D58; footprint LED_SMD:LED_0805_2012Metric_Pad1.15x1.40mm_HandSolder -> LED_SMD:LED_0201_0603Metric
- D6: renamed from D5; footprint LED_SMD:LED_0805_2012Metric_Pad1.15x1.40mm_HandSolder -> LED_SMD:LED_0201_0603Metric
- D60: renamed from D59; footprint LED_SMD:LED_0805_2012Metric_Pad1.15x1.40mm_HandSolder -> LED_SMD:LED_0201_0603Metric
- D61: renamed from D60; footprint LED_SMD:LED_0805_2012Metric_Pad1.15x1.40mm_HandSolder -> LED_SMD:LED_0201_0603Metric
- D62: renamed from D61; footprint LED_SMD:LED_0805_2012Metric_Pad1.15x1.40mm_HandSolder -> LED_SMD:LED_0201_0603Metric
- D63: renamed from D62; footprint LED_SMD:LED_0805_2012Metric_Pad1.15x1.40mm_HandSolder -> LED_SMD:LED_0201_0603Metric
- D64: renamed from D63; footprint LED_SMD:LED_0805_2012Metric_Pad1.15x1.40mm_HandSolder -> LED_SMD:LED_0201_0603Metric
- D65: renamed from D64; footprint LED_SMD:LED_0805_2012Metric_Pad1.15x1.40mm_HandSolder -> LED_SMD:LED_0201_0603Metric
- D7: renamed from D6; footprint LED_SMD:LED_0805_2012Metric_Pad1.15x1.40mm_HandSolder -> LED_SMD:LED_0201_0603Metric
- D8: renamed from D7; footprint LED_SMD:LED_0805_2012Metric_Pad1.15x1.40mm_HandSolder -> LED_SMD:LED_0201_0603Metric
- D9: renamed from D8; footprint LED_SMD:LED_0805_2012Metric_Pad1.15x1.40mm_HandSolder -> LED_SMD:LED_0201_0603Metric
- renumbered U3 to U2
Connections:
- net +3.3V: now also C17.1, C18.1, U3.23 (VCC)
- net GND: now also C17.2, C18.2, C19.2, R12.2, R13.2, U3.24 (GND), U3.28 (AD), U3.33 (GND), U3.9 (GND)
- net LEDMTX.C0: now also U3.30 (CS1)
- net LEDMTX.C1: now also U3.31 (CS2)
- net LEDMTX.C2: now also U3.32 (CS3)
- net LEDMTX.C3: now also U3.1 (CS4)
- net LEDMTX.C4: now also U3.2 (CS5)
- net LEDMTX.C5: now also U3.3 (CS6)
- net LEDMTX.C6: now also U3.4 (CS7)
- net LEDMTX.C7: now also U3.5 (CS8)
- net LEDMTX.R0: now also U3.22 (SW1)
- net LEDMTX.R1: now also U3.21 (SW2)
- net LEDMTX.R2: now also U3.20 (SW3)
- net LEDMTX.R3: now also U3.19 (SW4)
- net LEDMTX.R4: now also U3.18 (SW5)
- net LEDMTX.R5: now also U3.17 (SW6)
- net LEDMTX.R6: now also U3.16 (SW7)
- net LEDMTX.R7: now also U3.15 (SW8)
- new net: R12.1, U3.25 (ISET)
- new net I2C.SCL: U3.27 (SCL)
- new net I2C.SDA: U3.26 (SDA)
- new net ~{MX_SDB}: C19.1, R13.1, U3.29 (~{SDB})
- no-connect marks 0 -> 8
Other:
- company: (none) -> George Sleen

Commit message: Switch THT IR components to SMD ones
Parts:
- removed U2: TLC59116, Package_SO:TSSOP-28_4.4x9.7mm_P0.65mm, symbol GS_IC:TLC59116
- renumbered C18 to C17, C17 to C18, D7 to D10, D8 to D11, D9 to D12, D10 to D13, D11 to D14, D12 to D15, D13 to D16, D14 to D17, D15 to D18, D16 to D19, D17 to D20, D18 to D21, D19 to D22, D20 to D23, D21 to D24, D22 to D25, D23 to D26, D24 to D27, D25 to D28, D26 to D29, D27 to D30, D28 to D31, D29 to D32, D30 to D33, D31 to D34, D32 to D35, D33 to D36, D34 to D37, D35 to D38, D36 to D39, D37 to D40, D38 to D41, D39 to D42, D40 to D43, D41 to D44, D42 to D45, D43 to D46, D44 to D47, D45 to D48, D46 to D49, D2 to D5, D47 to D50, D48 to D51, D49 to D52, D50 to D53, D51 to D54, D52 to D55, D53 to D56, D54 to D57, D55 to D58, D56 to D59, D3 to D6, D57 to D60, D58 to D61, D59 to D62, D60 to D63, D61 to D64, D62 to D65, D63 to D66, D64 to D67, D65 to D68, D4 to D7, D5 to D8, D6 to D9, R13 to R12, R12 to R13, U3 to U6

Commit message: Draft layout
Parts:
- removed C17: 4.7uF, Capacitor_SMD:C_0402_1005Metric, symbol Device:C
- renumbered C19 to C18, C18 to C20, D45 to D10, D53 to D11, D61 to D12, D6 to D13, D22 to D15, D30 to D16, D38 to D17, D46 to D18, D54 to D19, D62 to D20, D7 to D21, D15 to D22, D31 to D24, D39 to D25, D47 to D26, D55 to D27, D63 to D28, D8 to D29, D16 to D30, D24 to D31, D40 to D33, D48 to D34, D56 to D35, D64 to D36, D9 to D37, D17 to D38, D25 to D39, D33 to D40, D49 to D42, D57 to D43, D65 to D44, D10 to D45, D18 to D46, D26 to D47, D34 to D48, D42 to D49, D58 to D51, D66 to D52, D11 to D53, D19 to D54, D27 to D55, D35 to D56, D43 to D57, D51 to D58, D13 to D6, D67 to D60, D12 to D61, D20 to D62, D28 to D63, D36 to D64, D44 to D65, D52 to D66, D60 to D67, D21 to D7, D29 to D8, D37 to D9, R12 to R14, U6 to U5

Commit message: Finish Silkscreen
Parts:
- C18, C20: footprint Capacitor_SMD:C_0201_0603Metric -> GS_SMD:0201_0603Metric
- D10, D11, D12, D13, D14, D15, D16, D17, D18, D19, D20, D21, D22, D23, D24, D25, D26, D27, D28, D29, D30, D31, D32, D33, D34, D35, D36, D37, D38, D39, D40, D41, D42, D43, D44, D45, D46, D47, D48, D49, D5, D50, D51, D52, D53, D54, D55, D56, D57, D58, D59, D6, D60, D61, D62, D63, D64, D65, D66, D67, D68, D7, D8, D9: footprint LED_SMD:LED_0201_0603Metric -> GS_Optoelectronics:LED_0201_0603Metric
- R13, R14: footprint Resistor_SMD:R_0201_0603Metric -> GS_SMD:0201_0603Metric
