File: microcouple/capacitive-touch.kicad_sch (KiCad schematic)
At the start: 6 parts, among them J4 Conn_02x03_Odd_Even, U6 CAP1188

Commit message: Change all components to 0402 if smaller
Parts:
- C21, C22: footprint GS_Capacitors:C_0201_0603Metric -> GS_Capacitors:C_0402_1005Metric; symbol GS_Capacitor_0201:C_0201_100nF -> GS_Capacitor_0402:C_0402_100nF; LCSC ID C18164587 -> C344189; Mfr. Part # TCC0201X5R104M250ZT -> TCC0402X5R104K160AT; Package 0201 -> 0402
- R15: footprint GS_Resistors:R_0201_0603Metric -> GS_Resistors:R_0402_1005Metric; symbol GS_Resistor_0201:R_0201_10k -> GS_Resistor_0402:R_0402_10k; LCSC ID C304504 -> C102759; Manufacturer FH (Guangdong Fenghua Advanced Tech) -> RALEC; Mfr. Part # RC-01W103JT -> RTT02103JTH; Package 0201 -> 0402
- R16: footprint GS_Resistors:R_0201_0603Metric -> GS_Resistors:R_0402_1005Metric; symbol GS_Resistor_0201:R_0201_100k -> GS_Resistor_0402:R_0402_100k; LCSC ID C106224 -> C3017514; Manufacturer YAGEO -> VO; Mfr. Part # RC0201FR-07100KL -> SCR0402J100K; Package 0201 -> 0402
