File: microcouple/ir-transciever.kicad_sch (KiCad schematic)
At the start: 4 parts, among them U7 IRM-V838M3-C/TR1

Commit message: Change all components to 0402 if smaller
Parts:
- C23: footprint GS_Capacitors:C_0201_0603Metric -> GS_Capacitors:C_0402_1005Metric; symbol GS_Capacitor_0201:C_0201_100nF -> GS_Capacitor_0402:C_0402_100nF; LCSC ID C18164587 -> C344189; Mfr. Part # TCC0201X5R104M250ZT -> TCC0402X5R104K160AT; Package 0201 -> 0402
- R17: footprint GS_Resistors:R_0201_0603Metric -> GS_Resistors:R_0402_1005Metric; symbol GS_Resistor_0201:R_0201_330R -> GS_Resistor_0402:R_0402_330R; LCSC ID C320833 -> C2906929; Manufacturer FH (Guangdong Fenghua Advanced Tech) -> FOJAN; Mfr. Part # RC-01W3300FT -> FRC0402J331 TS; Package 0201 -> 0402
Changed lines of the file:
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@@
 	)
 	(symbol
-		(lib_id "GS_Capacitor_0201:C_0201_100nF")
+		(lib_id "GS_Capacitor_0402:C_0402_100nF")
 		(at 63.5 68.58 0)
 		(unit 1)
@@
 			)
 		)
-		(property "Footprint" "GS_Capacitors:C_0201_0603Metric"
-			(at 64.4652 72.39 0)
+		(property "Footprint" "GS_Capacitors:C_0402_1005Metric"
+			(at 63.5 46.228 0)
 			(effects
 				(font
@@
 			)
 		)
-		(property "Datasheet" "https://www.lcsc.com/datasheet/lcsc_datasheet_2410121315_CCTC-TCC0201X5R104M250ZT_C18164587.pdf"
-			(at 63.5 68.58 0)
+		(property "Datasheet" "https://www.lcsc.com/datasheet/lcsc_datasheet_2410121315_CCTC-TCC0402X5R104K160AT_C344189.pdf"
+			(at 63.5 54.864 0)
 			(effects
 				(font
@@
 			)
 		)
-		(property "Description" "Unpolarized capacitor"
-			(at 63.5 68.58 0)
+		(property "Description" "100nF 10% Unpolarized Capacitor, 16V Max Voltage, X5R"
+			(at 63.5 52.832 0)
 			(effects
 				(font
@@
 		)
 		(property "Manufacturer" "CCTC"
-			(at 63.5 68.58 0)
+			(at 63.5 49.53 0)
 			(effects
 				(font
@@
 			)
 		)
-		(property "Package" "0201"
-			(at 63.5 68.58 0)
+		(property "Package" "0402"
+			(at 63.5 48.006 0)
 			(effects
 				(font
@@
 			)
 		)
-		(property "LCSC ID" "C18164587"
-			(at 63.5 68.58 0)
+		(property "LCSC ID" "C344189"
+			(at 63.5 56.642 0)
 			(effects
 				(font
@@
 			)
 		)
-		(property "Mfr. Part #" "TCC0201X5R104M250ZT"
-			(at 63.5 68.58 0)
+		(property "Mfr. Part #" "TCC0402X5R104K160AT"
+			(at 63.5 51.308 0)
 			(effects
 				(font
@@
 	)
 	(symbol
-		(lib_id "GS_Resistor_0201:R_0201_330R")
+		(lib_id "GS_Resistor_0402:R_0402_330R")
 		(at 121.92 74.93 0)
 		(unit 1)
@@
 			)
 		)
-		(property "Footprint" "GS_Resistors:R_0201_0603Metric"
+		(property "Footprint" "GS_Resistors:R_0402_1005Metric"
 			(at 121.92 52.832 0)
 			(effects
@@
 			)
 		)
-		(property "Datasheet" "https://www.lcsc.com/datasheet/lcsc_datasheet_2411121005_FH--Guangdong-Fenghua-Advanced-Tech-RC-01W3300FT_C320833.pdf"
-			(at 121.92 57.404 0)
+		(property "Datasheet" "https://www.lcsc.com/datasheet/lcsc_datasheet_2411071710_FOJAN-FRC0402J331-TS_C2906929.pdf"
+			(at 121.92 55.372 0)
 			(effects
 				(font
@@
 			)
 		)
-		(property "Description" "Resistor, US symbol"
-			(at 121.92 48.26 0)
+		(property "Description" "330R 5% Resistor, 62.5mW Max Power, 50V Max Voltage, 100ppm"
+			(at 122.174 48.006 0)
 			(effects
 				(font
@@
 			)
 		)
-		(property "Manufacturer" "FH (Guangdong Fenghua Advanced Tech)"
-			(at 121.92 55.118 0)
+		(property "Manufacturer" "FOJAN"
+			(at 121.92 59.944 0)
 			(effects
 				(font
@@
 			)
 		)
-		(property "Mfr. Part #" "RC-01W3300FT"
-			(at 121.92 50.292 0)
+		(property "Mfr. Part #" "FRC0402J331 TS"
+			(at 121.92 50.546 0)
 			(effects
 				(font
@@
 			)
 		)
-		(property "LCSC ID" "C320833"
+		(property "LCSC ID" "C2906929"
 			(at 121.92 46.228 0)
 			(effects
@@
 			)
 		)
-		(property "Package" "0201"
-			(at 121.92 44.45 0)
+		(property "Package" "0402"
+			(at 121.92 57.912 0)
 			(effects
 				(font
