File: microcouple/microcouple.kicad_sch (KiCad schematic)
At the start: 34 parts, among them J1 Conn_ARM_SWD_TagConnect_TC203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, J2 USB_C_Socket, SW1 SW_Push, U1 USBLC6-2P6-MS, U2 RP2040, X1 12MHz 12pF

Commit message: Change missing part on JLC
Parts:
- U1: symbol GS_IC:USBLC6-2P6-MS -> GS_IC:USBLC6-2P6; LCSC ID C3647099 -> C2827693; Manufacturer MSKSEMI -> TECH PUBLIC; Mfr. Part # USBLC6-2P6-MS -> USBLC6-2P6; Package SOT-666 -> SOT-666-6
Changed lines of the file:
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@@
 	)
 	(symbol
-		(lib_id "GS_IC:USBLC6-2P6-MS")
+		(lib_id "GS_IC:USBLC6-2P6")
 		(at 78.74 78.74 0)
 		(unit 1)
@@
 			)
 		)
-		(property "Datasheet" "https://www.lcsc.com/datasheet/lcsc_datasheet_2501211645_MSKSEMI-USBLC6-2P6-MS_C3647099.pdf"
+		(property "Datasheet" "https://www.lcsc.com/datasheet/lcsc_datasheet_2411121100_TECH-PUBLIC-USBLC6-2P6_C2827693.pdf"
 			(at 79.756 87.376 0)
 			(effects
@@
 			)
 		)
-		(property "Manufacturer" "MSKSEMI"
+		(property "Manufacturer" "TECH PUBLIC"
 			(at 78.74 62.23 0)
 			(effects
@@
 			)
 		)
-		(property "Mfr. Part #" "USBLC6-2P6-MS"
+		(property "Mfr. Part #" "USBLC6-2P6"
 			(at 78.74 56.134 0)
 			(effects
@@
 			)
 		)
-		(property "LCSC ID" "C3647099"
+		(property "LCSC ID" "C2827693"
 			(at 78.74 58.166 0)
 			(effects
@@
 			)
 		)
-		(property "Package" "SOT-666"
+		(property "Package" "SOT-666-6"
 			(at 78.74 60.198 0)
 			(effects

Commit message: Change all components to 0402 if smaller
Parts:
- C10, C12, C19, C2, C24, C25, C26, C5, C6, C7: footprint GS_Capacitors:C_0201_0603Metric -> GS_Capacitors:C_0402_1005Metric; symbol GS_Capacitor_0201:C_0201_100nF -> GS_Capacitor_0402:C_0402_100nF; LCSC ID C18164587 -> C344189; Mfr. Part # TCC0201X5R104M250ZT -> TCC0402X5R104K160AT; Package 0201 -> 0402
- C3, C4: footprint GS_Capacitors:C_0201_0603Metric -> GS_Capacitors:C_0402_1005Metric; symbol GS_Capacitor_0201:C_0201_14pF -> GS_Capacitor_0402:C_0402_14pF; LCSC ID C3037637 -> C3037644; Mfr. Part # 0201CG140J500NT -> 0402CG140J500NT; Package 0201 -> 0402
- D1: footprint GS_Optoelectronics:LED_0201_0603Metric -> GS_Optoelectronics:LED_0402_1005Metric; symbol GS_Optoelectronic:LED_0201_Green -> GS_Optoelectronic:LED_0402_Green; LCSC ID C3646922 -> C965793; Mfr. Part # XL-0201UGC -> XL-1005UGC; Package 0201 -> 0402
- R1, R2, R6, R7, R8: footprint GS_Resistors:R_0201_0603Metric -> GS_Resistors:R_0402_1005Metric; symbol GS_Resistor_0201:R_0201_5.1k -> GS_Resistor_0402:R_0402_5.1k; LCSC ID C158467 -> C453708; Manufacturer RALEC -> FH (Guangdong Fenghua Advanced Tech); Mfr. Part # RTT01512JTH -> RC-02K512JT; Package 0201 -> 0402
- R3: footprint GS_Resistors:R_0201_0603Metric -> GS_Resistors:R_0402_1005Metric; symbol GS_Resistor_0201:R_0201_1k -> GS_Resistor_0402:R_0402_1k; LCSC ID C304503 -> C2906899; Manufacturer FH (Guangdong Fenghua Advanced Tech) -> FOJAN; Mfr. Part # RC-01W102JT -> FRC0402J102 TS; Package 0201 -> 0402
