File: pcb/ir-transciever.kicad_sch (KiCad schematic)
At the start: 4 parts, among them U7 IRM-V838M3-C/TR1

Commit message: Prepare schematic for revision 2.0.0
Parts:
- D69: footprint easyeda2kicad:LED-SMD_L3.0-W2.7-RD -> GS_Optoelectronics:LED_SMD_L3.0-W2.7-RD
- U7: footprint easyeda2kicad:OPTO-SMD_IRM-V838M3-C-TR1 -> GS_Optoelectronics:IRM-V8__M3-C-TR1
Changed lines of the file:
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@@
 		(title "IR Transciever")
 		(date "2025-04-27")
-		(rev "A")
+		(rev "2.0.0")
 		(company "George Sleen")
 	)
@@
 			)
 		)
-		(property "Footprint" "easyeda2kicad:OPTO-SMD_IRM-V838M3-C-TR1"
+		(property "Footprint" "GS_Optoelectronics:IRM-V8__M3-C-TR1"
 			(at 81.28 88.9 0)
 			(effects
@@
 				)
 				(hide yes)
-			)
-		)
-		(property "LCSC Part" ""
-			(at 81.28 77.47 0)
-			(effects
-				(font
-					(size 1.27 1.27)
-				)
 			)
 		)
@@
 			)
 		)
-		(property "Footprint" "easyeda2kicad:LED-SMD_L3.0-W2.7-RD"
+		(property "Footprint" "GS_Optoelectronics:LED_SMD_L3.0-W2.7-RD"
 			(at 110.236 59.69 0)
 			(effects
@@
 				)
 				(hide yes)
-			)
-		)
-		(property "LCSC Part" ""
-			(at 121.92 59.69 0)
-			(effects
-				(font
-					(size 1.27 1.27)
-				)
 			)
 		)
@@
 			)
 		)
-		(property "LCSC Part" ""
-			(at 63.5 68.58 0)
-			(effects
-				(font
-					(size 1.27 1.27)
-				)
-			)
-		)
 		(pin "1"
 		)
@@
 			)
 		)
-		(property "LCSC Part" ""
-			(at 121.92 74.93 0)
-			(effects
-				(font
-					(size 1.27 1.27)
-				)
-			)
-		)
