File: pcb/microcouple.kicad_pcb (KiCad board)
At the start: 4 copper layers, 29.5 x 34.2 mm, 133 parts, among them J1 Conn_ARM_SWD_TagConnect_TC203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, J2 USB_C_Socket, J4 Conn_02x03_Odd_Even, Q1 AO3415, SW1 SW_Push, SW2 MSK12CO2, U1 USBLC6-2P6-MS, U2 RP2040, U3 MCP73831, U4 AP63203WU-7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

Commit message: Prepare schematic for revision 2.0.0
Parts:
- added C28: 100nF, GS_Capacitors:C_0402_1005Metric, F.Cu at (18.1, 27.0)
- added U8: W25Q128JVSIQ, GS_SO:SOIC-8_5.3x5.3mm_P1.27mm, F.Cu at (21.8, 22.6)
- D69: footprint easyeda2kicad:LED-SMD_L3.0-W2.7-RD -> GS_Optoelectronics:LED_SMD_L3.0-W2.7-RD
- U7: footprint easyeda2kicad:OPTO-SMD_IRM-V838M3-C-TR1 -> GS_Optoelectronics:IRM-V8__M3-C-TR1
Connections:
- SW2 pad 2: /Battery Management/VIN -> GND
- U2 pad 51: unconnected-(U2-QSPI_SD3-Pad51) -> /EEPROM/QSPI.IO3
- U2 pad 52: unconnected-(U2-QSPI_SCLK-Pad52) -> /EEPROM/QSPI.SCK
- U2 pad 53: unconnected-(U2-QSPI_SD0-Pad53) -> /EEPROM/QSPI.IO0
- U2 pad 54: unconnected-(U2-QSPI_SD2-Pad54) -> /EEPROM/QSPI.IO2
- U2 pad 55: unconnected-(U2-QSPI_SD1-Pad55) -> /EEPROM/QSPI.IO1
- U2 pad 56: unconnected-(U2-QSPI_SS-Pad56) -> /QSPI.~{CS}
